File: devboard/DevBoard.sch (KiCad schematic (older format))
At the start: 7 parts, among them J1 J2, J2 J3, U1 74HC573, U2 74HC573, U3 IS62WV12816ALL, U4 74HC573, U5 74HC573

Commit message: Added Flash
Parts:
- added U1: OscillatorSocket, Package_DIP:DIP-14_W7.62mm_Socket, symbol DevBoard:OscillatorSocket
- added U6, U7: 74HC245, Package_DIP:DIP-20_W7.62mm, symbol 74xx:74HC245
- added U9: S29AL008J70TFI013, Package_SO:TSOP-I-48_18.4x12mm_P0.5mm, symbol DevBoard:S29AL008J70TFI013
- U2: renamed from U4; footprint Package_DIP:DIP-20_W7.62mm_Socket -> Package_DIP:DIP-20_W7.62mm
- U3: renamed from U1; footprint Package_DIP:DIP-20_W7.62mm_Socket -> Package_DIP:DIP-20_W7.62mm
- U4: renamed from U2; footprint Package_DIP:DIP-20_W7.62mm_Socket -> Package_DIP:DIP-20_W7.62mm
- U5: footprint Package_DIP:DIP-20_W7.62mm_Socket -> Package_DIP:DIP-20_W7.62mm
- renumbered U3 to U8
Connections:
- net A4: now reaches U2.15 (Q4), U8.1 (A4)
- net A4: now also U9.21 (A4)
- net IO3: now reaches U8.10 (I/O3)
- net IO3: now also U6.5 (A3), U9.35 (DQ3)
- net 3.3V: now reaches J1.38 (Pin_38), U8.11 (VDD), U8.33 (VDD)
- net 3.3V: now also U2.20 (VCC), U3.20 (VCC), U4.20 (VCC), U5.20 (VCC), U6.20 (VCC), U7.20 (VCC), U9.12 (RESET), U9.14 (WP), U9.37 (Vcc), U9.47 (BYTE)
- net GND: now reaches J2.40 (Pin_40), U2.1 (OE), U2.10 (GND), U3.1 (OE), U3.10 (GND), U4.1 (OE), U4.10 (GND), U5.1 (OE), U5.10 (GND), U8.12 (GND), U8.34 (GND)
- net GND: now also U8.41 (OE), U1.7 (GND), U6.10 (GND), U7.10 (GND), U9.27 (GND), U9.28 (OE), U9.46 (GND)
- net IO4: now reaches U8.13 (I/O4)
- net IO4: now also U6.6 (A4), U9.38 (DQ4)
- net IO5: now reaches U8.14 (I/O5)
- net IO5: now also U6.7 (A5), U9.40 (DQ5)
- net IO6: now reaches U8.15 (I/O6)
- net IO6: now also U6.8 (A6), U9.42 (DQ6)
- net IO7: now reaches U8.16 (I/O7)
- net IO7: now also U6.9 (A7), U9.44 (DQ7)
- net WE: now reaches U8.17 (WE)
- net WE: now also J2.38 (Pin_38), U6.1 (A->B), U7.1 (A->B), U9.11 (WE)
- net A16: now reaches U8.18 (A16)
- net A16: now also U4.19 (Q0), U9.48 (A16)
- net A15: now reaches U8.19 (A15)
- net A15: now also U3.12 (Q7), U9.1 (A15); no longer U5.12 (Q7)
- net A3: now reaches U2.16 (Q3), U8.2 (A3)
- net A3: now also U9.22 (A3)
- net A14: now reaches U8.20 (A14)
- net A14: now also U3.13 (Q6), U9.2 (A14); no longer U5.13 (Q6)
- net A13: now reaches U8.21 (A13)
- net A13: now also U3.14 (Q5), U9.3 (A13); no longer U5.14 (Q5)
- net A12: now reaches U8.22 (A12)
- net A12: now also U3.15 (Q4), U9.4 (A12); no longer U5.15 (Q4)
- net A11: now reaches U8.24 (A11)
- net A11: now also U3.16 (Q3), U9.5 (A11); no longer U5.16 (Q3)
- net A10: now reaches U8.25 (A10)
- net A10: now also U3.17 (Q2), U9.6 (A10); no longer U5.17 (Q2)
- net A25: now reaches U5.18 (Q1)
- net A25: no longer U8.26 (A9)
- net A24: now reaches U5.19 (Q0)
- net A24: no longer U8.27 (A8)
- net IO8: now reaches U8.29 (I/O8)
- net IO8: now also U7.2 (A0), U9.30 (DQ8)
- net A2: now reaches U2.17 (Q2), U8.3 (A2)
- net A2: now also U9.23 (A2)
- net IO9: now reaches U8.30 (I/O9)
- net IO9: now also U7.3 (A1), U9.32 (DQ9)
- net IO10: now reaches U8.31 (I/O10)
- net IO10: now also U7.4 (A2), U9.34 (DQ10)
- net IO11: now reaches U8.32 (I/O11)
- net IO11: now also U7.5 (A3), U9.36 (DQ11)
- net IO12: now reaches U8.35 (I/O12)
- net IO12: now also U7.6 (A4), U9.39 (DQ12)
- net IO13: now reaches U8.36 (I/O13)
- net IO13: now also U7.7 (A5), U9.41 (DQ13)
- net IO14: now reaches U8.37 (I/O14)
- net IO14: now also U7.8 (A6), U9.43 (DQ14)
- net IO15: now reaches U8.38 (I/O15)
- net IO15: now also U7.9 (A7), U9.45 (DQ15)
- net A0: now reaches U8.39 (LB)
- net A0: now also U2.19 (Q0), U8.5 (A0), U9.25 (A0)
- net A1: now reaches U2.18 (Q1), U8.4 (A1)
- net A1: now also U9.24 (A1)
- net BHE: now reaches U8.40 (UB)
- net BHE: now also J2.3 (Pin_3)
- net A7: now reaches U2.12 (Q7), U8.42 (A7)
- net A7: now also U9.18 (A7)
- net A6: now reaches U2.13 (Q6), U8.43 (A6)
- net A6: now also U9.19 (A6)
- net A5: now reaches U2.14 (Q5), U8.44 (A5)
- net A5: now also U9.20 (A5)
- net A31: now reaches U8.6 (CS1)
- net A31: now also U5.12 (Q7)
- net IO0: now reaches U8.7 (I/O0)
- net IO0: now also U6.2 (A0), U9.29 (DQ0)
- net IO1: now reaches U8.8 (I/O1)
- net IO1: now also U6.3 (A1), U9.31 (DQ1)
- net IO2: now reaches U8.9 (I/O2)
- net IO2: now also U6.4 (A2), U9.33 (DQ2)
- net ALE1: now reaches J2.36 (Pin_36), U4.11 (Load)
- net ALE1: now also U5.11 (Load); no longer U3.11 (Load)
- net A9: now reaches U3.18 (Q1)
- net A9: now also U8.26 (A9), U9.7 (A9)
- net A8: now reaches U3.19 (Q0)
- net A8: now also U8.27 (A8), U9.8 (A8)
- net D0: now reaches J2.2 (Pin_2), U2.2 (D0)
- net D0: now also U4.2 (D0), U6.18 (B0); no longer U3.2 (D0)
- net D1: now reaches J2.4 (Pin_4), U2.3 (D1)
- net D1: now also U4.3 (D1), U6.17 (B1); no longer U3.3 (D1)
- net D2: now reaches J2.6 (Pin_6), U2.4 (D2)
- net D2: now also U4.4 (D2), U6.16 (B2); no longer U3.4 (D2)
- net D3: now reaches J2.8 (Pin_8), U2.5 (D3)
- net D3: now also U4.5 (D3), U6.15 (B3); no longer U3.5 (D3)
- net D4: now reaches J2.10 (Pin_10), U2.6 (D4)
- net D4: now also U4.6 (D4), U6.14 (B4); no longer U3.6 (D4)
- net D5: now reaches J2.12 (Pin_12), U2.7 (D5)
- net D5: now also U4.7 (D5), U6.13 (B5); no longer U3.7 (D5)
- net D6: now reaches J2.14 (Pin_14), U2.8 (D6)
- net D6: now also U4.8 (D6), U6.12 (B6); no longer U3.8 (D6)
- net D7: now reaches J2.16 (Pin_16), U2.9 (D7)
- net D7: now also U4.9 (D7), U6.11 (B7); no longer U3.9 (D7)
- net A23: now reaches U4.12 (Q7)
- net A22: now reaches U4.13 (Q6)
- net A21: now reaches U4.14 (Q5)
- net A20: now reaches U4.15 (Q4)
- net A19: now reaches U4.16 (Q3)
- net A18: now reaches U4.17 (Q2)
- net A18: now also U9.16 (A18)
- net A17: now reaches U4.18 (Q1)
- net A17: now also U9.17 (A17)
- net D8: now reaches J2.18 (Pin_18), U5.2 (D0)
- net D8: now also U3.2 (D0), U7.18 (B0); no longer U4.2 (D0)
- net D9: now reaches J2.20 (Pin_20), U5.3 (D1)
- net D9: now also U3.3 (D1), U7.17 (B1); no longer U4.3 (D1)
- net D10: now reaches J2.22 (Pin_22), U5.4 (D2)
- net D10: now also U3.4 (D2), U7.16 (B2); no longer U4.4 (D2)
- net D11: now reaches J2.24 (Pin_24), U5.5 (D3)
- net D11: now also U3.5 (D3), U7.15 (B3); no longer U4.5 (D3)
- net D12: now reaches J2.26 (Pin_26), U5.6 (D4)
- net D12: now also U3.6 (D4), U7.14 (B4); no longer U4.6 (D4)
- net D13: now reaches J2.28 (Pin_28), U5.7 (D5)
- net D13: now also U3.7 (D5), U7.13 (B5); no longer U4.7 (D5)
- net D14: now reaches J2.30 (Pin_30), U5.8 (D6)
- net D14: now also U3.8 (D6), U7.12 (B6); no longer U4.8 (D6)
- net D15: now reaches J2.32 (Pin_32), U5.9 (D7)
- net D15: now also U3.9 (D7), U7.11 (B7); no longer U4.9 (D7)
- net ALE0: now reaches J2.34 (Pin_34), U2.11 (Load)
- net ALE0: now also U3.11 (Load); no longer U5.11 (Load)
- net OE: now reaches J2.1 (Pin_1)
- net OE: now also U6.19 (CE), U7.19 (CE)
- net CLK: now reaches J2.5 (Pin_5)
- net CLK: now also U1.1 (OUT)
- new net 5V: J2.39 (Pin_39), U1.14 (Vcc)
- new net A26: U5.17 (Q2)
- new net A27: U5.16 (Q3)
- new net A28: U5.15 (Q4)
- new net A29: U5.14 (Q5)
- new net A30: U5.13 (Q6), U9.26 (CE)
- no-connect marks 99 -> 61
Other:
- moved on the sheet: U4, U8

Commit message: Board modifications
Parts:
- removed J1: J2, Connector_PinSocket_2.54mm:PinSocket_2x20_P2.54mm_Vertical, symbol DevBoard:J2
- removed J2: J3, Connector_PinSocket_2.54mm:PinSocket_2x20_P2.54mm_Vertical, symbol DevBoard:J3
- added C1, C2, C3, C4, C5, C6: 0.1u, symbol Device:C
- added C7, C8: C, symbol Device:C
- added M1: icewerx, devboard:iceWerx, symbol DevBoard:icewerx
- U2, U3, U4, U5, U6, U7: footprint Package_DIP:DIP-20_W7.62mm -> Package_SO:SOIC-20W_7.5x12.8mm_P1.27mm
- U8: Note (none) -> SRAM
- U9: Note (none) -> FRAM
Connections:
- net 3.3V: no longer U2.20 (VCC), U3.20 (VCC), U4.20 (VCC), U5.20 (VCC), U6.20 (VCC), U7.20 (VCC)
- net ALE0: no longer U2.11 (Load)
- net D0: no longer U2.2 (D0), U4.2 (D0)
- net D1: no longer U2.3 (D1), U4.3 (D1)
- net D10: no longer U3.4 (D2), U5.4 (D2)
- net D11: no longer U3.5 (D3), U5.5 (D3)
- net D12: no longer U3.6 (D4), U5.6 (D4)
- net D13: no longer U3.7 (D5), U5.7 (D5)
- net D14: no longer U3.8 (D6), U5.8 (D6)
- net D15: no longer U3.9 (D7), U5.9 (D7)
- net D2: no longer U2.4 (D2), U4.4 (D2)
- net D3: no longer U2.5 (D3), U4.5 (D3)
- net D4: no longer U2.6 (D4), U4.6 (D4)
- net D5: no longer U2.7 (D5), U4.7 (D5)
- net D6: no longer U2.8 (D6), U4.8 (D6)
- net D7: no longer U2.9 (D7), U4.9 (D7)
- net D8: no longer U3.2 (D0), U5.2 (D0)
- net D9: no longer U3.3 (D1), U5.3 (D1)
- net GND: now also C1.2, C2.2, C3.2, C4.2, C5.2, C6.2, C7.2, C8.2; no longer U2.1 (OE)
- net IO0: now also U2.2 (D0), U4.2 (D0), M1.J2.30 (B1)
- net IO1: now also U2.3 (D1), U4.3 (D1), M1.J2.28 (D3)
- net IO10: now also U3.4 (D2), U5.4 (D2), M1.J2.29 (C3)
- net IO11: now also U3.5 (D3), U5.5 (D3), M1.J2.27 (C1)
- net IO12: now also U3.6 (D4), U5.6 (D4), M1.J2.25 (E1)
- net IO13: now also U3.7 (D5), U5.7 (D5), M1.J2.23 (G1)
- net IO14: now also U3.8 (D6), U5.8 (D6), M1.J2.21 (H1)
- net IO15: now also U3.9 (D7), U5.9 (D7), M1.J2.19 (J1)
- net IO2: now also U2.4 (D2), U4.4 (D2), M1.J2.26 (D1)
- net IO3: now also U2.5 (D3), U4.5 (D3), M1.J2.24 (F3)
- net IO4: now also U2.6 (D4), U4.6 (D4), M1.J2.22 (G3)
- net IO5: now also U2.7 (D5), U4.7 (D5), M1.J2.20 (H3)
- net IO6: now also U2.8 (D6), U4.8 (D6), M1.J2.18 (J3)
- net IO7: now also U2.9 (D7), U4.9 (D7), M1.J2.16 (L1)
- net IO8: now also U3.2 (D0), U5.2 (D0), M1.J2.14 (N1)
- net IO9: now also U3.3 (D1), U5.3 (D1), M1.J2.12 (P1)
- net 5V: no longer names the net of U1.14 (Vcc)
- new net +3V3: C1.1, C2.1, C3.1, C4.1, C5.1, C6.1, C7.1, C8.1, U2.20 (VCC), U3.20 (VCC), U4.20 (VCC), U5.20 (VCC), U6.20 (VCC), U7.20 (VCC)
- no-connect marks 61 -> 6
Other:
- note added: "*Look into UART"
- note added: "Data bus latch"
- note added: "Data/Address bus header"
- note added: "External connector for clock source\n\nMultiple on-board clock sources."
- note added: "Female header socket for all of the FPGA pins"
- note added: "Keystone 5015 testpoint"
- note added: "Pin breakout\nLEDs\nPushbuttons\n"
- note added: "i2c and SPI peripheral"
- note added: "iceWerx board headers"
- moved on the sheet: U1, U2, U3, U4, U5, U6, U7, U8, U9
